Commit message: ready for ontology

File: urdf/robot_assignment.xacro (robot description, xacro)
@@ -1,245 +1,233 @@
-<?xml version="1.0"?>
-<robot xmlns:xacro="http://www.ros.org/wiki/xacro" name="robot_assignment_xacro">
-<!--To optimize the code it remains to make the progrma to compute the inertia of each link-->
-	<xacro:include filename="$(find robot_urdf)/urdf/materials.xacro" />
-	<xacro:include filename="$(find robot_urdf)/urdf/robot_assignment.gazebo" />
-	<xacro:property name="length_wheel" value="0.04" />
-	<xacro:property name="radius_wheel" value="0.08" />
-	<xacro:property name="arm_link_length" value="0.15" />
-	<xacro:property name="arm_link_radius" value="0.05" />
-	<xacro:macro name="default_inertial" params="mass">
-			<inertial>
-				<mass value="${mass}" />
-				<origin rpy="0 1.5707 1.5707" xyz="0 0 0"/>
-				<inertia ixx="0.000526666666667" ixy="0" ixz="0" iyy="0.000526666666667" iyz="0" izz="0.001"/>
-			</inertial>
-	</xacro:macro>
-	<xacro:macro name="cylinder_inertia" params="mass r l">
-			<inertia ixx="${mass*(3*r*r+l*l)/12}" ixy = "0" ixz = "0" iyy="${mass*(3*r*r+l*l)/12}" iyz = "0" izz="${mass*(r*r)/2}" />
- 	</xacro:macro>
-	<xacro:macro name="wheel_geometry">
-	<geometry>
-		<cylinder length="${length_wheel}" radius="${radius_wheel}"/>
-	</geometry>
-	</xacro:macro>
-	<xacro:macro name="arm_link_geometry">
-	<geometry>
-		<cylinder length="${arm_link_length}" radius="${arm_link_radius}"/>
-	</geometry>
-	</xacro:macro>
-	<!--Macro for robot's link-->
-	<xacro:macro name="link_wheel" params="name">
-		<link name="${name}">
-			<inertial>
-				<mass value="0.2"/>
-				<origin rpy="0 1.5707 1.5707" xyz="0 0 0"/>
-				<inertia ixx="0.000526666666667" ixy="0" ixz="0" iyy="0.000526666666667" iyz="0" izz="0.001"/>
-			</inertial>
-			<collision name="${name}_collision">
-				<origin rpy="0 1.5707 1.5707" xyz="0 0 0"/>
-				<geometry>
-					<cylinder length="0.04" radius="0.1"/>
-				</geometry>
-			</collision>
-			<visual name="${name}_visual">
-				<origin rpy="0 1.5707 1.5707" xyz="0 0 0"/>
-				<geometry>
-					<cylinder length="0.04" radius="0.1"/>
-				</geometry>
-			</visual>
-		</link>
-	</xacro:macro>
-	<xacro:macro name="arm_base_link" params="name ">
-		<link name="${name}">
-			<inertial>
-				<mass value="0.2"/>
-				<origin rpy="0 0 0" xyz="0 0 0"/>
-				<inertia ixx="0.000208333333333" ixy="0" ixz="0" iyy="0.000208333333333" iyz="0" izz="0.008333333333333"/>
-			</inertial>
-			<collision name="arm_base_link_collision">
-				<origin rpy="0 0 0" xyz="0 0 0"/>
-				<geometry>
-					<box size="0.1 0.1 0.05"/>
-				</geometry>
-			</collision>
-			<visual name="arm_base_link_visual">
-				<origin rpy="0 0 0" xyz="0 0 0"/>
-				<geometry>
-					<box size="0.1 0.1 0.05"/>
-				</geometry>
-			</visual>
-		</link>
-	</xacro:macro>
-	<xacro:macro name="arm_link" params="name ">
+<?xml version="1.0" ?>
+<robot name="m2wr" xmlns:xacro="https://www.ros.org/wiki/xacro" >
+  <xacro:include filename="$(find inspection_robot)/urdf/materials.xacro" />
+  <xacro:include filename="$(find inspection_robot)/urdf/robot_assignment.gazebo" />
+  <xacro:macro name="cylinder_inertia" params="mass r l">
+    <inertia ixx="${mass*(3*r*r+l*l)/12}" ixy = "0" ixz = "0"
+    iyy="${mass*(3*r*r+l*l)/12}" iyz = "0" izz="${mass*(r*r)/2}" />
+  </xacro:macro>
+  <xacro:macro name="link_wheel" params="name">
+    <link name="${name}">
+      <inertial>
+        <mass value="0.2"/>
+        <origin rpy="0 1.5707 1.5707" xyz="0 0 0"/>
+      <inertia ixx="0.000526666666667" ixy="0" ixz="0" iyy="0.000526666666667" iyz="0" izz="0.001"/>
+      </inertial>
+      <collision name="link_right_wheel_collision">
+        <origin rpy="0 1.5707 1.5707" xyz="0 0 0"/>
+        <geometry>
+          <cylinder length="0.04" radius="0.1"/>
+        </geometry>
+      </collision>
+      <visual name="${name}_visual">
+        <origin rpy="0 1.5707 1.5707" xyz="0 0 0"/>
+        <geometry>
+          <cylinder length="0.04" radius="0.1"/>
+        </geometry>
+      </visual>
+    </link>
+  </xacro:macro>
+  <xacro:macro name="arm_link" params="name arm_link_length xyz_origin">
 		<link name="${name}">
 			<inertial>
 				<origin xyz="0 0 0" rpy="0 0 0"/>
 				<mass value="0.025"/>
-				<xacro:cylinder_inertia mass="0.025" r="0.05" l="0.15"/>
+				<inertia ixx="0.000010279" ixy="0" ixz="0" iyy="0.000010279" iyz="0" izz="0.000007225"/>
 			</inertial>
 			<collision name="${name}_collision">
-				<origin rpy="0 0 0" xyz="0 0 0.075"/>
-				<xacro:arm_link_geometry />
+				<origin rpy="0 0 0" xyz="${xyz_origin}"/>
+        <geometry>
+          <cylinder length="${arm_link_length}" radius="0.04"/>
+        </geometry>
 			</collision>
 			<visual name="${name}_visual">
-				<origin rpy="0 0 0" xyz="0 0 0.075"/>
-				<xacro:arm_link_geometry />
+				<origin rpy="0 0 0" xyz="${xyz_origin}"/>
+        <geometry>
+          <cylinder length="${arm_link_length}" radius="0.04"/>
+        </geometry>
 			</visual>
 		</link>
 	</xacro:macro>
-	<!--Macro for robot's joint-->
-	<xacro:macro name="continuous_joint" params="name child parent origin_xyz axis_xyz">
-		<joint name="${name}" type="continuous">
-			<origin rpy="0 0 0" xyz="${origin_xyz}"/>
-			<child link="${child}"/>
-			<parent link="${parent}"/>
-			<axis rpy="0 0 0" xyz="${axis_xyz}"/>
-			<limit effort="10000" velocity="1000"/>
-			<joint_properties damping="1.0" friction="1.0"/>
-		</joint>
-	</xacro:macro>
-	<xacro:macro name="revolute_joint" params="name child parent origin_xyz">
-		<joint name="${name}" type="revolute">
-			<origin rpy="0 0 0" xyz="${origin_xyz}"/>
-			<child link="${child}"/>
-			<parent link="${parent}"/>
-			<axis rpy="0 0 0" xyz="1 0 0"/>
-			<limit effort="100.0" upper = "1.5" lower = "-1.5" velocity="0.5"/>
-			<joint_properties damping="1.0" friction="1.0"/>
-		</joint>
-	</xacro:macro>
-	<link name="link_chassis">
-		<!-- pose and inertial -->
-		<pose>0 0 0.1 0 0 0</pose>
-		<inertial>
-			<mass value="5"/>
-			<origin rpy="0 0 0" xyz="0 0 0.1"/>
-			<inertia ixx="0.0395416666667" ixy="0" ixz="0" iyy="0.106208333333" iyz="0" izz="0.106208333333"/>
-		</inertial>
-		<!-- body -->
-		<collision name="collision_chassis">
-			<geometry>
-				<box size="0.5 0.3 0.07"/>
-			</geometry>
-		</collision>
-		<visual>
-			<origin rpy="0 0 0" xyz="0 0 0"/>
-			<geometry>
-				<box size="0.5 0.3 0.07"/>
-			</geometry>
-			<material name="blue"/>
-		</visual>
-		<!-- caster front -->
-		<collision name="caster_front_collision">
-			<origin rpy=" 0 0 0" xyz="0.35 0 -0.05"/>
-			<geometry>
-				<sphere radius="0.05"/>
-			</geometry>
-			<surface>
-				<friction>
-					<ode>
-						<mu>0</mu>
-						<mu2>0</mu2>
-						<slip1>1.0</slip1>
-						<slip2>1.0</slip2>
-					</ode>
-				</friction>
-			</surface>
-		</collision>
-		<visual name="caster_front_visual">
-			<origin rpy=" 0 0 0" xyz="0.2 0 -0.05"/>
-			<geometry>
-				<sphere radius="0.05"/>
-			</geometry>
-		</visual>
-	</link>
-	<xacro:link_wheel name="right_wheel_link"/>
-	<xacro:link_wheel name="left_wheel_link"/>
-	<!-- Here put rìthe arm base link xacro-->
-	<xacro:arm_base_link name="arm_base_link"/>
-	<xacro:arm_link name="arm_1_link"/>
-	<xacro:arm_link name="arm_2_link"/>
-	<xacro:arm_link name="arm_3_link"/>
-	<link name="camera_link">
-	<inertial>
-		<mass value="1e-5" />
-		<origin xyz="0 0 0" rpy="0 0 0"/>
-		<inertia ixx="1e-6" ixy="0" ixz="0" iyy="1e-6" iyz="0" izz="1e-6" />
-	</inertial>
-	<collision>
-		<origin xyz="0 0 0.025" rpy="0 0 0"/>
-		<geometry>
-			<box size="0.15 0.1 0.05"/>
-		</geometry>
-	</collision>
-	<visual>
-		<origin xyz="0 0 0.025" rpy="0 0 0"/>
-		<geometry>
-			<box size="0.15 0.1 0.05"/>
-		</geometry>
-		<material name="red">
-		<color rgba="1 0 0 1"/>
-		</material>
-	</visual>
-	</link>
-	<!-- ####Definition of all the robot joints#### -->
-	<!-- Wheel joints -->
-	<xacro:continuous_joint name="right_wheel_joint"   child="right_wheel_link"  parent="link_chassis"  origin_xyz="-0.05 0.15 0"  axis_xyz="0 1 0"/>
-	<xacro:continuous_joint name="left_wheel_joint"   child="left_wheel_link"   parent="link_chassis"  origin_xyz="-0.05 -0.15 0"  axis_xyz="0 1 0"/>
-	<!-- Arm base link joint -->
-	<xacro:continuous_joint name="arm_base_joint"   child="arm_base_link"  parent="link_chassis"  origin_xyz="0 0 0.06"  axis_xyz="0 0 1" />
-	<!-- Arm link joints -->
-	<xacro:revolute_joint name="base_to_arm_1_joint"   child="arm_1_link"  parent="arm_base_link"  origin_xyz="0 0 0.025"/>
-	<xacro:revolute_joint name="arm_1_to_arm_2_joint"   child="arm_2_link"  parent="arm_1_link"  origin_xyz="0 0 0.15"/>
-	<xacro:revolute_joint name="arm_2_to_arm_3_joint"   child="arm_3_link"  parent="arm_2_link"  origin_xyz="0 0 0.15"/>
-	<!--Camera link joint -->
-	<joint name="camera_to_arm_3_joint" type="fixed">
-		<origin rpy="0 0 0" xyz="0 0 0.15"/>
-		<child link="camera_link"/>
-		<parent link="arm_3_link"/>
-		<axis rpy="0 0 0" xyz="0 1 0"/>
-		<limit effort="100.0" upper = "1.5" lower = "-1.5" velocity="0.5"/>
-		<joint_properties damping="1.0" friction="1.0"/>
+  <xacro:macro name="joint_wheel" params="name child origin_xyz">
+    <joint name="${name}" type="continuous">
+      <origin rpy="0 0 0" xyz="${origin_xyz}"/>
+      <child link="${child}"/>
+      <parent link="base_link"/>
+      <axis rpy="0 0 0" xyz="0 1 0"/>
+      <limit effort="10000" velocity="1000"/>
+      <joint_properties damping="1.0" friction="1.0"/>
+    </joint>
+  </xacro:macro>
+  <xacro:macro name="revolute_joint" params="name parent child origin_xyz axis_xyz">
+    <joint name="${name}" type="revolute">
+      <axis xyz="${axis_xyz}"/>
+      <limit effort="1000.0" lower="-3.14" upper="3.14" velocity="0.02"/>
+      <origin rpy="0 0 0" xyz="${origin_xyz}"/>
+      <parent link="${parent}"/>
+      <child link="${child}"/>
+    </joint>
+  </xacro:macro>
+  <link name="base_link">
+    <!-- pose and inertial -->
+    <pose>0 0 0.1 0 0 0</pose>
+    <inertial>
+      <mass value="5"/>
+      <origin rpy="0 0 0" xyz="0 0 0.1"/>
+      <inertia ixx="0.0395416666667" ixy="0" ixz="0" iyy="0.106208333333" iyz="0" izz="0.106208333333"/>
+    </inertial>
+    <collision name="collision_chassis">
+      <geometry>
+      <box size="0.5 0.3 0.07"/>
+      </geometry>
+    </collision>
+    <visual>
+      <origin rpy="0 0 0" xyz="0 0 0"/>
+      <geometry>
+        <box size="0.5 0.3 0.07"/>
+      </geometry>
+      <material name="blue"/>
+    </visual>
+      <!-- caster front -->
+    <collision name="caster_front_collision">
+      <origin rpy=" 0 0 0" xyz="0.35 0 -0.05"/>
+      <geometry>
+        <sphere radius="0.05"/>
+      </geometry>
+      <surface>
+        <friction>
+          <ode>
+            <mu>0</mu>
+            <mu2>0</mu2>
+            <slip1>1.0</slip1>
+            <slip2>1.0</slip2>
+          </ode>
+        </friction>
+      </surface>
+    </collision>
+    <visual name="caster_front_visual">
+      <origin rpy=" 0 0 0" xyz="0.2 0 -0.05"/>
+      <geometry>
+        <sphere radius="0.05"/>
+      </geometry>
+    </visual>
+  </link>
+  <!-- Create wheels -->
+  <xacro:link_wheel name="link_right_wheel" />
+  <xacro:link_wheel name="link_left_wheel" />
+  <xacro:joint_wheel name="joint_right_wheel"  child="link_right_wheel"  origin_xyz="-0.05 0.15 0"  />
+  <xacro:joint_wheel name="joint_left_wheel"   child="link_left_wheel"   origin_xyz="-0.05 -0.15 0"  />
+  <link name="laser">
+    <inertial>
+      <origin xyz="0 0 0" rpy="0 0 0" />
+      <mass value="1" />
+      <xacro:cylinder_inertia mass="1" r="0.05" l="0.1" />
+    </inertial>
+    <visual>
+      <origin xyz="0 0 0" rpy="0 0 0" />
+      <geometry>
+        <cylinder radius="0.05" length="0.1"/>
+      </geometry>
+      <material name="white" />
+    </visual>
+    <collision>
+      <origin xyz="0 0 0" rpy="0 0 0"/>
+      <geometry>
+        <cylinder radius="0.05" length="0.1"/>
+      </geometry>
+    </collision>
+  </link>
+  <joint name="joint_laser" type="fixed">
+    <origin xyz="0.15 0 0.05" rpy="0 0 0"/>
+    <parent link="base_link"/>
+    <child link="laser"/>
+  </joint>
+<!--arm definition -->
+  <link name="arm_base_link">
+  	<inertial>
+  		<mass value="0.1"/>
+  		<origin xyz="0 0 0" rpy="0 0 0" />
+  		<inertia ixx="0.0000416666667" ixy="0" ixz="0" iyy="0.0000416666667" iyz="0" izz="0.0000416666667"/>
+  	</inertial>
+  	<collision>
+  	  <origin xyz="0 0 0" rpy="0 0 0"/>
+      <geometry>
+        <box size="0.1 0.1 0.1"/>
+      </geometry>
+  	</collision>
+  	<visual>
+  	  <origin xyz="0 0 0" rpy="0 0 0"/>
+      <geometry>
+        <box size="0.1 0.1 0.1"/>
+      </geometry>
+      <material name="red" />
+  	</visual>
+  </link>
+  <joint name="arm_base_to_base" type="fixed">
+  	<origin rpy="0 0 0" xyz="0 0 0.05"/>
+  	<parent link="base_link"/>
+  	<child link="arm_base_link"/>
+  </joint>
+  <xacro:arm_link name="arm_link_01" arm_link_length="0.15" xyz_origin="0 0 0.075"/>
+  <xacro:arm_link name="arm_link_02" arm_link_length="0.15" xyz_origin="0 0 0.075"/>
+  <xacro:arm_link name="arm_link_03" arm_link_length="0.06" xyz_origin="0 0 0.03"/>
+  <xacro:revolute_joint name="arm_joint_01" child="arm_link_01" parent="arm_base_link" origin_xyz="0 0 0.025" axis_xyz="0 0 1"/>
+  <xacro:revolute_joint name="arm_joint_02" child="arm_link_02" parent="arm_link_01" origin_xyz="0 0 0.15" axis_xyz="1 0 0"/>
+  <xacro:revolute_joint name="arm_joint_03" child="arm_link_03" parent="arm_link_02" origin_xyz="0 0 0.15" axis_xyz="0 1 0"/>
+    <link name="camera_link">
+  	<inertial>
+  		<mass value="0.025"/>
+  		<origin xyz="0 0 0" rpy="0 0 0" />
+  		<inertia ixx="0.000010279" ixy="0" ixz="0" iyy="0.000010279" iyz="0" izz="0.000007225"/>
+  	</inertial>
+  	<collision>
+  	  <origin xyz="0 0 0" rpy="0 0 0"/>
+      <geometry>
+        <box size="0.08 0.08 0.08"/>
+      </geometry>
+  	</collision>
+  	<visual>
+  	  <origin xyz="0 0 0" rpy="0 0 1.57"/>
+      <geometry>
+        <box size="0.08 0.08 0.08"/>
+      </geometry>
+      <material name="red" >
+        <color rgba="1 0 0 1"/>
+      </material>
+  	</visual>
+  </link>
+  <joint name="camera_joint" type="fixed">
+  	<origin rpy="0 0 0" xyz="0 0 0.1"/>
+  	<parent link="arm_link_03"/>
+  	<child link="camera_link"/>
+  </joint>
+<transmission name="arm_joint_01_trans">
+	<type>transmission_interface/SimpleTransmission</type>
+	<joint name="arm_joint_01">
+		<hardwareInterface>hardware_interface/EffortJointInterface</hardwareInterface>
 	</joint>
-	<!-- Transmissions -->
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
Commit message: move base added

File: urdf/robot_assignment.xacro (robot description, xacro)
@@ -138,5 +138,5 @@
   </link>
   <joint name="joint_laser" type="fixed">
-    <origin xyz="0.15 0 0.05" rpy="0 0 0"/>
+    <origin xyz="0.30 0 0.05" rpy="0 0 0"/>
     <parent link="base_link"/>
     <child link="laser"/>
